File: prototype_schematics/LMR14050SDDA_reference/LMR14050SDDA_reference.sch (KiCad schematic (older format))
At the start: 49 parts, among them J1 USB_C_Receptacle_USB2.0, J10 USB_C_Receptacle_USB2.0, J2 Conn_EN, J3 ground holes, J4 V_in alt, J5 V_out alt, J6 DC_in, J7 Conn_EN, J8 V_in alt, J9 V_out alt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

Commit message: Final changes for ordering.
Parts:
- R7, R8: value R -> 3.3k
Changed lines of the file:
@@
 P 7800 2250
 F 0 "R7" H 7870 2296 50  0000 L CNN
-F 1 "R" H 7870 2205 50  0000 L CNN
+F 1 "3.3k" H 7870 2205 50  0000 L CNN
 F 2 "Resistor_SMD:R_0805_2012Metric" V 7730 2250 50  0001 C CNN
 F 3 "~" H 7800 2250 50  0001 C CNN
@@
 P 8400 2250
 F 0 "R8" H 8470 2296 50  0000 L CNN
-F 1 "R" H 8470 2205 50  0000 L CNN
+F 1 "3.3k" H 8470 2205 50  0000 L CNN
 F 2 "Resistor_SMD:R_0805_2012Metric" V 8330 2250 50  0001 C CNN
 F 3 "~" H 8400 2250 50  0001 C CNN

Commit message: Change USB C receptacle to a component that's in stock.
Parts:
- J1, J10: footprint Connector_USB:USB_C_Receptacle_GCT_USB4085 -> Connector_USB:USB_C_Receptacle_HRO_TYPE-C-31-M-12
Changed lines of the file:
@@
 F 0 "J1" H 10207 4667 50  0000 C CNN
 F 1 "USB_C_Receptacle_USB2.0" H 10207 4576 50  0000 C CNN
-F 2 "Connector_USB:USB_C_Receptacle_GCT_USB4085" H 10250 3800 50  0001 C CNN
+F 2 "Connector_USB:USB_C_Receptacle_HRO_TYPE-C-31-M-12" H 10250 3800 50  0001 C CNN
 F 3 "https://www.usb.org/sites/default/files/documents/usb_type-c.zip" H 10250 3800 50  0001 C CNN
 	1    10100 3800
@@
 F 0 "J10" H 10207 7317 50  0000 C CNN
 F 1 "USB_C_Receptacle_USB2.0" H 10207 7226 50  0000 C CNN
-F 2 "Connector_USB:USB_C_Receptacle_GCT_USB4085" H 10250 6450 50  0001 C CNN
+F 2 "Connector_USB:USB_C_Receptacle_HRO_TYPE-C-31-M-12" H 10250 6450 50  0001 C CNN
 F 3 "https://www.usb.org/sites/default/files/documents/usb_type-c.zip" H 10250 6450 50  0001 C CNN
 	1    10100 6450
